Commit message: update hexapod_description

File: software/hexapod_ros_ws/src/hexapod_description/urdf/hexapod_description.urdf (robot description, URDF)
Before this commit: robot hexapod_description, 21 links, 20 joints
Joints:
- joint tibia1_joint: limit lower=-0.7854 upper=3.1416 effort=0 velocity=0 -> lower=-0.7854 upper=2.09 effort=0 velocity=0
- joint tibia2_joint: limit lower=-0.7854 upper=3.1416 effort=0 velocity=0 -> lower=-0.7854 upper=2.09 effort=0 velocity=0
- joint tibia3_joint: limit lower=-0.7854 upper=3.1416 effort=0 velocity=0 -> lower=-0.7854 upper=2.09 effort=0 velocity=0
- joint tibia4_joint: limit lower=-0.7854 upper=3.1416 effort=0 velocity=0 -> lower=-0.7854 upper=2.09 effort=0 velocity=0
- joint tibia5_joint: limit lower=-0.7854 upper=3.1416 effort=0 velocity=0 -> lower=-0.7854 upper=2.09 effort=0 velocity=0
- joint tibia6_joint: limit lower=-0.7854 upper=3.1416 effort=0 velocity=0 -> lower=-0.7854 upper=2.09 effort=0 velocity=0

Commit message: rename lidar_link to laser_frame

File: software/hexapod_ros_ws/src/hexapod_description/urdf/hexapod_description.urdf (robot description, URDF)
Before this commit: robot hexapod_description, 21 links, 20 joints
Links:
- removed link lidar_link
- added link laser_frame, mass 0.0387549710715716; collision mesh filename=package://hexapod_description/meshes/laser_frame.STL; visual mesh filename=package://hexapod_description/meshes/laser_frame.STL
Joints:
- joint lidar_joint: child lidar_link -> laser_frame
- joint tibia1_joint: limit lower=-0.7854 upper=2.09 effort=0 velocity=0 -> lower=-2.09 upper=1.06 effort=0 velocity=0
- joint tibia2_joint: limit lower=-0.7854 upper=2.09 effort=0 velocity=0 -> lower=-2.09 upper=1.06 effort=0 velocity=0
- joint tibia3_joint: limit lower=-0.7854 upper=2.09 effort=0 velocity=0 -> lower=-2.09 upper=1.06 effort=0 velocity=0
- joint tibia4_joint: limit lower=-0.7854 upper=2.09 effort=0 velocity=0 -> lower=-2.09 upper=1.06 effort=0 velocity=0
- joint tibia5_joint: limit lower=-0.7854 upper=2.09 effort=0 velocity=0 -> lower=-2.09 upper=1.06 effort=0 velocity=0
- joint tibia6_joint: limit lower=-0.7854 upper=2.09 effort=0 velocity=0 -> lower=-2.09 upper=1.06 effort=0 velocity=0
